Commit message: Tidy up code: ABB IRB120.

File: ABBRobots/IRB120/irb120_ros2_gazebo/urdf/irb120.urdf.xacro (robot description, xacro)
@@ -48,12 +48,126 @@
 -->
 <robot name="irb120" xmlns:xacro="http://ros.org/wiki/xacro">
+  <!-- ===== ARGUMENTS ===== -->
+  <!-- CELL LAYOUT:  -->
+  <xacro:arg name="cell_layout_1" default="false"/>
+  <xacro:property name="cell_layout_1" value="$(arg cell_layout_1)"/>
+  <xacro:arg name="cell_layout_2" default="false"/>
+  <xacro:property name="cell_layout_2" value="$(arg cell_layout_2)"/>
+  <xacro:arg name="cell_layout_3" default="false"/>
+  <xacro:property name="cell_layout_3" value="$(arg cell_layout_3)"/>
+  <!-- END-EFFECTOR:  -->
+  <xacro:arg name="EE_no" default="false"/>
+  <xacro:property name="EE_no" value="$(arg EE_no)"/>
+  <xacro:arg name="EE_schunk" default="false"/>
+  <xacro:property name="EE_schunk" value="$(arg EE_schunk)"/>
   <!-- Include XACRO-MACRO file of the IRB120: -->
   <xacro:include filename="$(find irb120_ros2_gazebo)/urdf/irb120_macro.urdf.xacro"/>
-  <xacro:irb120 prefix=""/>
-  <!-- Fix robot to Gazebo world -->
+  <xacro:irb120
+    prefix=""
+    EE_no="${EE_no}"
+    EE_schunk="${EE_schunk}"
+  />
+  <!-- Gazebo WORLD link: -->
   <link name="world"/>
-  <joint name="world-base_link-fixed" type="fixed">
-    <parent link="world"/>
-    <child link="base_link"/>
-  </joint>
+  <!-- ========== ========== ========== ========== ========== ========== -->
+  <!-- CELL LAYOUT SELECTION: -->
+  <!-- CELL LAYOUT N1) ABB IRB120 Robot alone: -->
+  <xacro:if value="${cell_layout_1}">
+    <joint name="world-base_link-fixed" type="fixed">
+      <parent link="world"/>
+      <child link="base_link"/>
+    </joint>
+  </xacro:if>
+  <!-- CELL LAYOUT N2) ABB IRB120 Robot in Cranfield University cell: -->
+  <xacro:if value="${cell_layout_2}">
+    <link name="cell">
+      <visual>
+        <origin xyz="-0.21 -0.357 0.0" rpy="0 0 0" />
+        <geometry>
+          <mesh filename="file://$(find irb120_ros2_gazebo)/meshes/irb120_cell.dae" scale="1 1 1" />
+        </geometry>
+      </visual>
+      <collision>
+        <origin xyz="-0.21 -0.357 0.0" rpy="0 0 0" />
+        <geometry>
+          <mesh filename="file://$(find irb120_ros2_gazebo)/meshes/irb120_cell.dae" scale="1 1 1" />
+        </geometry>
+      </collision>
+      <inertial>
+        <mass value="1000.0"/>
+        <inertia ixx="500.0" ixy="500.0" ixz="500.0" iyy="500.0" iyz="500.0" izz="500.0" />
+      </inertial>
+    </link>
+    <joint name="world-cell-fixed" type="fixed">
+      <parent link="world"/>
+      <child link="cell"/>
+    </joint>
+    <joint name="cell-base_link-fixed" type="fixed">
+      <parent link="cell"/>
+      <child link="base_link"/>
+      <origin xyz="0.0 0.0 0.015" rpy="0.0 0.0 0.0" />
+    </joint>
+  </xacro:if>
+  <!-- CELL LAYOUT N3) ABB IRB120 + PICK & PLACE layout: -->
+  <xacro:if value="${cell_layout_3}">
+    <link name='irb120_block'>
+      <inertial>
+        <origin xyz="0 0 0" rpy="0 0 0"/>
+        <mass value="100"/>
+        <inertia ixx="0.01"  ixy="0"  ixz="0" iyy="0.01" iyz="0" izz="0.01" />
+      </inertial>
+      <collision name='collision'>
+        <origin xyz="0 0 0" rpy=" 0 0 0"/>
+        <geometry>
+          <box size = "0.2 0.2 0.5"/>
+        </geometry>
+      </collision>
+      <visual name='chassis_visual'>
+        <origin xyz="0 0 0" rpy=" 0 0 0"/>
+        <geometry>
+          <box size = "0.2 0.2 0.5"/>
+        </geometry>
+        <material name="red">
+          <color rgba="1 0 0 1"/>
+        </material>
+      </visual>
+    </link>
+    <joint name="world_joint" type="fixed">
+      <parent link="world" />
+      <child link = "irb120_block" />
+      <origin xyz="0.0 0.0 0.25" rpy="0.0 0.0 0.0" />
+    </joint>
+    <joint name="block-base" type="fixed">
+      <parent link="irb120_block" />
+      <child link = "base_link" />
+      <origin xyz="0.0 0.0 0.255" rpy="0.0 0.0 0.0" />
+    </joint>
+    <link name='table'>
+      <inertial>
+        <origin xyz="0 0 0" rpy="0 0 0"/>
+        <mass value="100"/>
+        <inertia ixx="0.01"  ixy="0"  ixz="0" iyy="0.01" iyz="0" izz="0.01" />
+      </inertial>
+      <collision name='collision'>
+        <origin xyz="0 0 0" rpy=" 0 0 0"/>
+        <geometry>
+          <box size = "0.5 1.0 0.7"/>
+        </geometry>
+      </collision>
+      <visual name='chassis_visual'>
+        <origin xyz="0 0 0" rpy=" 0 0 0"/>
+        <geometry>
+          <box size = "0.5 1.0 0.7"/>
+        </geometry>
+        <material name="black">
+          <color rgba="1 0 0 1"/>
+        </material>
+      </visual>
+    </link>
+    <joint name="table_world" type="fixed">
+      <parent link="world" />
+      <child link = "table" />
+      <origin xyz="0.7 0.0 0.35" rpy="0.0 0.0 0.0" />
+    </joint>
+  </xacro:if>
 </robot>

File: ABBRobots/IRB120/irb120_ros2_gazebo/urdf/irb120_macro.urdf.xacro (robot description, xacro)
@@ -50,14 +50,19 @@
   <!-- Include additional ABB-Resources/MATERIALS+COLOUR xacro files: -->
   <xacro:include filename="$(find irb120_ros2_gazebo)/urdf/abb_resources/common_materials.xacro"/>
-  <!-- Load TRANSMISSION file: -->
-  <xacro:include filename="$(find irb120_ros2_gazebo)/urdf/irb120_transmission.xacro" />
-  <!-- Load GAZEBO/ROS2_CONTROL file: -->
-  <xacro:include filename="$(find irb120_ros2_gazebo)/urdf/irb120_gazebo.xacro" />
   <!-- XACRO-MACRO of ABB-IRB120: -->
-  <xacro:macro name="irb120" params="prefix">
-    <!-- ABB-IRB120 TRANSMISSION: -->
-    <xacro:irb120_transmission prefix=""/>
-    <!-- ABB-IRB120 GAZEBO - ROS2_CONTROL: -->
-    <xacro:irb120_gazebo prefix=""/>
+  <xacro:macro name="irb120" params="prefix EE_no EE_schunk">
+    <!-- Load ABB IRB120 TRANSMISSION file: -->
+    <xacro:include filename="$(find irb120_ros2_gazebo)/urdf/irb120_transmission.xacro" />
+    <xacro:irb120_transmission
+      prefix=""
+      EE_schunk="${EE_schunk}"
+    />
+    <!-- Load ABB IRB120 ROS2_CONTROL file: -->
+    <xacro:include filename="$(find irb120_ros2_gazebo)/urdf/irb120_ros2control.xacro" />
+    <xacro:irb120_ros2control
+      prefix=""
+      EE_no="${EE_no}"
+      EE_schunk="${EE_schunk}"
+    />
     <!-- ***** ABB-IRB120 ROBOT .urdf SERIAL CHAIN ***** -->
     <!-- Link list: -->
@@ -294,4 +299,194 @@
       <child link="${prefix}tool0" />
     </joint>
+    <!-- =================================== -->
+    <!-- ========== END-EFFECTORS ========== -->
+    <!-- === SCHUNK EGP-64 GRIPPER === -->
+    <xacro:if value="${EE_schunk}">
+      <!-- Schunk coupler (LINK): -->
+      <link name="schunk_coupler">
+        <visual>
+          <geometry>
+            <mesh filename="file://$(find irb120_ros2_gazebo)/meshes/egp64/Schunk Gripper - ADAPTER.dae" />
+          </geometry>
+          <material name="flat_black"/>
+        </visual>
+        <collision>
+          <geometry>
+            <mesh filename="file://$(find irb120_ros2_gazebo)/meshes/egp64/Schunk Gripper - ADAPTER.dae" />
+          </geometry>
+        </collision>
+        <inertial>
+          <origin xyz="0 0 0" rpy="0 0 ${pi/4}" />
+          <mass value="0.001" />
+          <inertia ixx="0.001" ixy="0.0" ixz="0.0" iyy="0.001" iyz="0.0" izz="0.001"/>
+        </inertial>
+      </link>
+      <!-- Schunk coupler (JOINT): -->
+      <joint name="schunk_coupler_joint" type="fixed">
+        <origin xyz="0 0 0.001" rpy="0 0 ${pi/4}" />
+        <parent link="tool0"/>
+        <child link="schunk_coupler"/>
+      </joint>
+      <gazebo reference="schunk_coupler">
+        <mu1>0.9</mu1>
+        <mu2>0.9</mu2>
+        <material>Gazebo/FlatBlack</material>
+      </gazebo>
+      <link name="egp64_gripper_base_link">
+        <inertial>
+          <origin xyz="0 0 0" rpy="0 0 0" />
+          <mass value="0.005" />
+          <inertia ixx="0.001" ixy="0.0" ixz="0.0" iyy="0.001" iyz="0.0" izz="0.001"/>
+        </inertial>
+        <visual>
+          <geometry>
+            <mesh filename="file://$(find irb120_ros2_gazebo)/meshes/egp64/Schunk Gripper - BASE noAdapter.dae" />
+          </geometry>
+          <material name="blue">
+            <color rgba="0 0 1 1"/>
+          </material>
+        </visual>
+        <collision>
+          <geometry>
+            <mesh filename="file://$(find irb120_ros2_gazebo)/meshes/egp64/Schunk Gripper - BASE noAdapter.dae" />
+          </geometry>
+          <material name="blue"/>
+        </collision>
+      </link>
+      <joint name="egp64_coupler" type="fixed">
+        <parent link="schunk_coupler"/>
+        <child link="egp64_gripper_base_link"/>
+        <origin xyz="-0.03205 0.01812 0.02047" rpy="0 0 0" />
+      </joint>
+      <!-- LEFT FINGER BASE -->
+      <link name="egp64_finger_left_link">
+        <inertial>
+          <origin xyz="0.01483 -0.00782 0" rpy="0 0 0" />
+          <mass value="0.002" />
+          <inertia ixx="0.001" ixy="0.0" ixz="0.0" iyy="0.001" iyz="0.0" izz="0.001"/>
+        </inertial>
+        <visual>
+          <geometry>
+            <mesh filename="file://$(find irb120_ros2_gazebo)/meshes/egp64/Schunk Gripper - LEFT FINGER BASE.dae" />
+          </geometry>
+          <material name="black">
+            <color rgba="0 0 0 1"/>
+          </material>
+        </visual>
+        <collision>
+          <geometry>
+            <mesh filename="file://$(find irb120_ros2_gazebo)/meshes/egp64/Schunk Gripper - LEFT FINGER BASE.dae" />
+          </geometry>
+          <material name="black" />
+        </collision>
+      </link>
+      <joint name="egp64_finger_left_joint" type="prismatic" >
+        <parent link="egp64_gripper_base_link" />
+        <child link="egp64_finger_left_link" />
+        <limit effort="100" lower="-0.001" upper="0.04" velocity="0.2"/>
+        <origin xyz="0.01483 -0.00782 0" rpy="0 0 0" />
+        <axis xyz="-1 0 0" />
+      </joint>
+      <!-- LEFT FINGERTIP -->
+      <link name="egp64_fingertip_left_link">
+        <inertial>
+          <origin xyz="0.03869 -0.0005 0.00093" rpy="0 0 0" />
+          <mass value="0.001" />
+          <inertia ixx="0.001" ixy="0.0" ixz="0.0" iyy="0.001" iyz="0.0" izz="0.001"/>
+        </inertial>
+        <visual>
+          <geometry>
+            <mesh filename="file://$(find irb120_ros2_gazebo)/meshes/egp64/Schunk Gripper - LEFT FINGER.dae" />
+          </geometry>
+          <material name="silver">
+            <color rgba="0.8 0.8 0.8 1"/>
+          </material>
+        </visual>
+        <collision>
+          <geometry>
+            <mesh filename="file://$(find irb120_ros2_gazebo)/meshes/egp64/Schunk Gripper - LEFT FINGER.dae" />
+          </geometry>
+          <material name="black"/>
+        </collision>
+      </link>
+      <joint name="egp64_fingertip_left_joint" type="fixed" >
+        <parent link="egp64_finger_left_link" />
+        <child link="egp64_fingertip_left_link" />
+        <origin xyz="0.03869 -0.0005 0.00093" rpy="0 0 0"/>
+      </joint>
+      <!-- RIGHT FINGER BASE -->
+      <link name="egp64_finger_right_link">
+        <inertial>
+          <origin xyz="-0.0153 -0.00602 0" rpy="0 0 0" />
+          <mass value="0.002" />
+          <inertia ixx="0.001" ixy="0.0" ixz="0.0" iyy="0.001" iyz="0.0" izz="0.001"/>
+        </inertial>
+        <visual>
+          <geometry>
+            <mesh filename="file://$(find irb120_ros2_gazebo)/meshes/egp64/Schunk Gripper - RIGHT FINGER BASE.dae" />
+          </geometry>
+          <material name="black"/>
+        </visual>
+        <collision>
+          <geometry>
+            <mesh filename="file://$(find irb120_ros2_gazebo)/meshes/egp64/Schunk Gripper - RIGHT FINGER BASE.dae" />
+          </geometry>
+          <material name="black"/>
+        </collision>
+      </link>
+      <joint name="egp64_finger_right_joint" type="prismatic" >
+        <parent link="egp64_gripper_base_link" />
+        <child link="egp64_finger_right_link" />
+        <limit effort="100" lower="-0.001" upper="0.04" velocity="0.2"/>
+        <origin xyz="-0.0153 -0.00602 0" rpy="0 0 0" />
+        <axis xyz="1 0 0" />
+      </joint>
+      <!-- RIGHT FINGERTIP -->
+      <link name="egp64_fingertip_right_link">
+        <inertial>
+          <origin xyz="-0.01211 -0.00197 0.00093" rpy="0 0 0" />
+          <mass value="0.001" />
+          <inertia ixx="0.001" ixy="0.0" ixz="0.0" iyy="0.001" iyz="0.0" izz="0.001"/>
+        </inertial>
+        <visual>
+          <geometry>
+            <mesh filename="file://$(find irb120_ros2_gazebo)/meshes/egp64/Schunk Gripper - RIGHT FINGER.dae" />
+          </geometry>
+          <material name="silver" />
+        </visual>
+        <collision>
+          <geometry>
+            <mesh filename="file://$(find irb120_ros2_gazebo)/meshes/egp64/Schunk Gripper - RIGHT FINGER.dae" />
+          </geometry>
+          <material name="black"/>
+      </collision>
+      </link>
+      <joint name="egp64_fingertip_right_joint" type="fixed" >
+        <parent link="egp64_finger_right_link" />
+        <child link="egp64_fingertip_right_link" />
+        <origin xyz="-0.01211 -0.00197 0.00093" rpy="0 0 0"/>
+      </joint>
+      <!-- SMALL CUBE FOR GRIPPER PLUGIN -->
+      <link name="EE_egp64">
+        <inertial>
+          <origin xyz="0 0 0" rpy="0 0 0" />
+          <mass value="0.00001" />
+          <inertia ixx="0.001" ixy="0.0" ixz="0.0" iyy="0.001" iyz="0.0" izz="0.001"/>
+        </inertial>
+        <visual>
+          <geometry>
+            <box size= "0.001 0.001 0.001" />
+          </geometry>
+        </visual>
+      </link>
+      <joint name="EE_egp64_joint" type="prismatic" >
+        <parent link="egp64_gripper_base_link" />
+        <child link="EE_egp64" />
+        <limit effort="10000" lower="0.0" upper="0.0" velocity="0.0"/>
+        <axis xyz="1 0 0" />
+        <origin xyz="0.033 -0.018 0.15" rpy="0 0 0"/>
+      </joint>
+    </xacro:if>
+    <!-- === SCHUNK EGP-64 GRIPPER === -->
   </xacro:macro>
 </robot>

File: ABBRobots/IRB120/irb120_ros2_gazebo/urdf/irb120_ros2control.xacro (robot description, xacro)
@@ -48,12 +48,28 @@
 -->
 <robot xmlns:xacro="http://www.ros.org/wiki/xacro">
-  <xacro:macro name="irb120_gazebo" params="prefix" >
-    <gazebo>
-      <plugin filename="libgazebo_ros2_control.so" name="gazebo_ros2_control">
-        <robot_sim_type>gazebo_ros2_control/GazeboSystem</robot_sim_type>
-        <parameters>$(find irb120_ros2_gazebo)/config/irb120_controller.yaml</parameters>
-      </plugin>
-    </gazebo>
-    <ros2_control name="GazeboSystem" type="system">
+  <xacro:macro name="irb120_ros2control" params="prefix EE_no EE_schunk" >
+    <!-- ROS2_CONTROL tag name: -->
+    <xacro:property name="name" value="GazeboSystem"/>
+    <!-- ===== Gazebo ROS2_CONTROL plugin ===== -->
+    <!-- No End-Effector: -->
+    <xacro:if value="${EE_no}">
+      <gazebo>
+        <plugin filename="libgazebo_ros2_control.so" name="gazebo_ros2_control">
+          <robot_sim_type>gazebo_ros2_control/GazeboSystem</robot_sim_type>
+          <parameters>$(find irb120_ros2_gazebo)/config/irb120_controller.yaml</parameters>
+        </plugin>
+      </gazebo>
+    </xacro:if>
+    <!-- End-Effector -> SCHUNK EGP-64 GRIPPER: -->
+    <xacro:if value="${EE_schunk}">
+      <gazebo>
+        <plugin filename="libgazebo_ros2_control.so" name="gazebo_ros2_control">
+          <robot_sim_type>gazebo_ros2_control/GazeboSystem</robot_sim_type>
+          <parameters>$(find irb120_ros2_gazebo)/config/irb120egp64_controller.yaml</parameters>
+        </plugin>
+      </gazebo>
+    </xacro:if>
+    <!-- ========== ROS2 CONTROL ========== -->
+    <ros2_control name="${name}" type="system">
       <hardware>
         <plugin>gazebo_ros2_control/GazeboSystem</plugin>
@@ -143,4 +159,50 @@
         <state_interface name="effort"/>
       </joint>
+      <!-- =================================== -->
+      <!-- ========== END-EFFECTORS ========== -->
+      <!-- === SCHUNK EGP-64 GRIPPER === -->
+      <xacro:if value="${EE_schunk}">
+        <!-- egp64_finger_left_joint -->
+        <joint name="egp64_finger_left_joint">
+          <command_interface name="position">
+            <param name="min">-0.001</param>
+            <param name="max">0.04</param>
+          </command_interface>
+          <command_interface name="velocity">
+            <param name="min">-0.2</param>
+            <param name="max">0.2</param>
+          </command_interface>
+          <state_interface name="position"/>
+          <state_interface name="velocity"/>
+        </joint>
+        <!-- egp64_finger_right_joint -->
+        <joint name="egp64_finger_right_joint">
+          <command_interface name="position">
+            <param name="min">-0.001</param>
+            <param name="max">0.04</param>
+          </command_interface>
+          <command_interface name="velocity">
+            <param name="min">-0.2</param>
+            <param name="max">0.2</param>
+          </command_interface>
+          <state_interface name="position"/>
+          <state_interface name="velocity"/>
+        </joint>
+        <joint name="EE_egp64_joint">
+          <command_interface name="position">
+            <param name="min">0.0</param>
+            <param name="max">0.0</param>
+          </command_interface>
+          <command_interface name="velocity">
+            <param name="min">0.0</param>
+            <param name="max">0.0</param>
+          </command_interface>
+          <state_interface name="position">
+            <param name="initial_value">0.0</param>
+          </state_interface>
+          <state_interface name="velocity"/>
+        </joint>
+      </xacro:if>
+      <!-- === SCHUNK EGP-64 GRIPPER === -->
     </ros2_control>
     <gazebo reference="${prefix}base_link">
@@ -172,4 +234,25 @@
       <material>Gazebo/Orange</material>
     </gazebo>
+    <!-- =================================== -->
+    <!-- ========== END-EFFECTORS ========== -->
+    <!-- === SCHUNK EGP-64 GRIPPER === -->
+    <xacro:if value="${EE_schunk}">
+      <gazebo reference="egp64_gripper_base_link">
+        <selfCollide>false</selfCollide>
+      </gazebo>
+      <gazebo reference="egp64_finger_left_link">
+        <selfCollide>false</selfCollide>
+      </gazebo>
+      <gazebo reference="egp64_fingertip_left_link">
+        <selfCollide>false</selfCollide>
+      </gazebo>
+      <gazebo reference="egp64_finger_right_link">
+        <selfCollide>false</selfCollide>
+      </gazebo>
+      <gazebo reference="egp64_fingertip_right_link">
+        <selfCollide>false</selfCollide>
+      </gazebo>
+    </xacro:if>
+    <!-- === SCHUNK EGP-64 GRIPPER === -->
     <gazebo reference="end_effector_frame_fixed_joint">
       <preserveFixedJoint>true</preserveFixedJoint>

File: ABBRobots/IRB120/irb120_ros2_gazebo/urdf/irb120_transmission.xacro (robot description, xacro)
@@ -48,5 +48,5 @@
 -->
 <robot xmlns:xacro="http://wiki.ros.org/xacro">
-  <xacro:macro name="irb120_transmission" params="prefix">
+  <xacro:macro name="irb120_transmission" params="prefix EE_schunk">
     <transmission name="irb120_joint1_trans">
       <type>transmission_interface/SimpleTransmission</type>
@@ -103,4 +103,28 @@
       </actuator>
     </transmission>
+    <!-- =================================== -->
+    <!-- ========== END-EFFECTORS ========== -->
+    <!-- === SCHUNK EGP-64 GRIPPER === -->
+    <xacro:if value="${EE_schunk}">
+      <transmission name="egp64_left_finger_trans">
+        <type>transmission_interface/SimpleTransmission</type>
+        <joint name="egp64_finger_left_joint">
+          <hardwareInterface>hardware_interface/PositionJointInterface</hardwareInterface>
+        </joint>
+        <actuator name="egp64_left_finger_motor">
+          <mechanicalReduction>1</mechanicalReduction>
+        </actuator>
+      </transmission>
+      <transmission name="egp64_right_finger_trans">
+        <type>transmission_interface/SimpleTransmission</type>
+        <joint name="egp64_finger_right_joint">
+          <hardwareInterface>hardware_interface/PositionJointInterface</hardwareInterface>
+        </joint>
+        <actuator name="egp64_right_finger_motor">
+          <mechanicalReduction>1</mechanicalReduction>
+        </actuator>
+      </transmission>
+    </xacro:if>
+    <!-- === SCHUNK EGP-64 GRIPPER === -->
   </xacro:macro>
 </robot>
