Commit message: Adapt repository: Foxy -> Humble.

File: ABBRobots/IRB120/irb120_ros2_gazebo/urdf/irb120_macro.urdf.xacro (robot description, xacro)
@@ -230,5 +230,5 @@
       <limit effort="0" lower="-2.87979" upper="2.87979" velocity="4.36332"/>
       <axis xyz="0 0 1"/>
-      <dynamics damping="0.0" friction="0.0"/>
+      <dynamics damping="50.0" friction="1.0"/>
     </joint>
     <!-- joint_2 -->
@@ -239,5 +239,5 @@
       <limit effort="0" lower="-1.91986" upper="1.91986" velocity="4.36332"/>
       <axis xyz="0 1 0"/>
-      <dynamics damping="0.0" friction="0.0"/>
+      <dynamics damping="50.0" friction="1.0"/>
     </joint>
     <!-- joint_3 -->
@@ -248,5 +248,5 @@
       <limit effort="0" lower="-1.91986" upper="1.22173" velocity="4.36332"/>
       <axis xyz="0 1 0"/>
-      <dynamics damping="0.0" friction="0.0"/>
+      <dynamics damping="10.0" friction="1.0"/>
     </joint>
     <!-- joint_4 -->
@@ -257,5 +257,5 @@
       <limit effort="0" lower="-2.79253" upper="2.79253" velocity="5.58505"/>
       <axis xyz="1 0 0"/>
-      <dynamics damping="0.0" friction="0.0"/>
+      <dynamics damping="5.0" friction="1.0"/>
     </joint>
     <!-- joint_5 -->
@@ -266,5 +266,5 @@
       <limit effort="0" lower="-2.094395" upper="2.094395" velocity="5.58505"/>
       <axis xyz="0 1 0"/>
-      <dynamics damping="0.0" friction="0.0"/>
+      <dynamics damping="2.0" friction="1.0"/>
     </joint>
     <!-- joint_6 -->
@@ -275,5 +275,5 @@
       <limit effort="0" lower="-6.98132" upper="6.98132" velocity="7.33038"/>
       <axis xyz="1 0 0"/>
-      <dynamics damping="0.0" friction="0.0"/>
+      <dynamics damping="1.0" friction="1.0"/>
     </joint>
     <!-- end of joint list -->
@@ -307,11 +307,10 @@
         <visual>
           <geometry>
-            <mesh filename="file://$(find irb120_ros2_gazebo)/meshes/egp64/Schunk Gripper - ADAPTER.dae" />
-          </geometry>
-          <material name="flat_black"/>
-        </visual>
-        <collision>
-          <geometry>
-            <mesh filename="file://$(find irb120_ros2_gazebo)/meshes/egp64/Schunk Gripper - ADAPTER.dae" />
+            <mesh filename="file://$(find irb120_ros2_gazebo)/meshes/egp64/egp64_Adapter.dae" />
+          </geometry>
+        </visual>
+        <collision>
+          <geometry>
+            <mesh filename="file://$(find irb120_ros2_gazebo)/meshes/egp64/egp64_Adapter.dae" />
           </geometry>
         </collision>
@@ -331,5 +330,5 @@
         <mu1>0.9</mu1>
         <mu2>0.9</mu2>
-        <material>Gazebo/FlatBlack</material>
+        <material>Gazebo/Black</material>
       </gazebo>
       <link name="egp64_gripper_base_link">
@@ -341,5 +340,5 @@
         <visual>
           <geometry>
-            <mesh filename="file://$(find irb120_ros2_gazebo)/meshes/egp64/Schunk Gripper - BASE noAdapter.dae" />
+            <mesh filename="file://$(find irb120_ros2_gazebo)/meshes/egp64/egp64_BaseNoAdapter.dae" />
           </geometry>
           <material name="blue">
@@ -349,5 +348,5 @@
         <collision>
           <geometry>
-            <mesh filename="file://$(find irb120_ros2_gazebo)/meshes/egp64/Schunk Gripper - BASE noAdapter.dae" />
+            <mesh filename="file://$(find irb120_ros2_gazebo)/meshes/egp64/egp64_BaseNoAdapter.dae" />
           </geometry>
           <material name="blue"/>
@@ -368,5 +367,5 @@
         <visual>
           <geometry>
-            <mesh filename="file://$(find irb120_ros2_gazebo)/meshes/egp64/Schunk Gripper - LEFT FINGER BASE.dae" />
+            <mesh filename="file://$(find irb120_ros2_gazebo)/meshes/egp64/egp64_LeftFingerBase.dae" />
           </geometry>
           <material name="black">
@@ -376,5 +375,5 @@
         <collision>
           <geometry>
-            <mesh filename="file://$(find irb120_ros2_gazebo)/meshes/egp64/Schunk Gripper - LEFT FINGER BASE.dae" />
+            <mesh filename="file://$(find irb120_ros2_gazebo)/meshes/egp64/egp64_LeftFingerBase.dae" />
           </geometry>
           <material name="black" />
@@ -387,4 +386,5 @@
         <origin xyz="0.01483 -0.00782 0" rpy="0 0 0" />
         <axis xyz="-1 0 0" />
+        <dynamics damping="1.0" friction="1.0"/>
       </joint>
       <!-- LEFT FINGERTIP -->
@@ -397,5 +397,5 @@
         <visual>
           <geometry>
-            <mesh filename="file://$(find irb120_ros2_gazebo)/meshes/egp64/Schunk Gripper - LEFT FINGER.dae" />
+            <mesh filename="file://$(find irb120_ros2_gazebo)/meshes/egp64/egp64_LeftFinger.dae" />
           </geometry>
           <material name="silver">
@@ -405,5 +405,5 @@
         <collision>
           <geometry>
-            <mesh filename="file://$(find irb120_ros2_gazebo)/meshes/egp64/Schunk Gripper - LEFT FINGER.dae" />
+            <mesh filename="file://$(find irb120_ros2_gazebo)/meshes/egp64/egp64_LeftFinger.dae" />
           </geometry>
           <material name="black"/>
@@ -424,5 +424,5 @@
         <visual>
           <geometry>
-            <mesh filename="file://$(find irb120_ros2_gazebo)/meshes/egp64/Schunk Gripper - RIGHT FINGER BASE.dae" />
+            <mesh filename="file://$(find irb120_ros2_gazebo)/meshes/egp64/egp64_RightFingerBase.dae" />
           </geometry>
           <material name="black"/>
@@ -430,5 +430,5 @@
         <collision>
           <geometry>
-            <mesh filename="file://$(find irb120_ros2_gazebo)/meshes/egp64/Schunk Gripper - RIGHT FINGER BASE.dae" />
+            <mesh filename="file://$(find irb120_ros2_gazebo)/meshes/egp64/egp64_RightFingerBase.dae" />
           </geometry>
           <material name="black"/>
@@ -441,4 +441,5 @@
         <origin xyz="-0.0153 -0.00602 0" rpy="0 0 0" />
         <axis xyz="1 0 0" />
+        <dynamics damping="1.0" friction="1.0"/>
       </joint>
       <!-- RIGHT FINGERTIP -->
@@ -451,5 +452,5 @@
         <visual>
           <geometry>
-            <mesh filename="file://$(find irb120_ros2_gazebo)/meshes/egp64/Schunk Gripper - RIGHT FINGER.dae" />
+            <mesh filename="file://$(find irb120_ros2_gazebo)/meshes/egp64/egp64_RightFinger.dae" />
           </geometry>
           <material name="silver" />
@@ -457,5 +458,5 @@
         <collision>
           <geometry>
-            <mesh filename="file://$(find irb120_ros2_gazebo)/meshes/egp64/Schunk Gripper - RIGHT FINGER.dae" />
+            <mesh filename="file://$(find irb120_ros2_gazebo)/meshes/egp64/egp64_RightFinger.dae" />
           </geometry>
           <material name="black"/>
@@ -486,4 +487,5 @@
         <axis xyz="1 0 0" />
         <origin xyz="0.033 -0.018 0.15" rpy="0 0 0"/>
+        <dynamics damping="1.0" friction="1.0"/>
       </joint>
     </xacro:if>

Commit message: Remove FlatBlack color.

File: ABBRobots/IRB120/irb120_ros2_gazebo/urdf/irb120_macro.urdf.xacro (robot description, xacro)
@@ -309,5 +309,4 @@
             <mesh filename="file://$(find irb120_ros2_gazebo)/meshes/egp64/Schunk Gripper - ADAPTER.dae" />
           </geometry>
-          <material name="flat_black"/>
         </visual>
         <collision>
@@ -331,5 +330,5 @@
         <mu1>0.9</mu1>
         <mu2>0.9</mu2>
-        <material>Gazebo/FlatBlack</material>
+        <material>Gazebo/Black</material>
       </gazebo>
       <link name="egp64_gripper_base_link">

Commit message: Mesh visual dae fix for IRB120, IRB1200 and PandaRobot
Signed-off-by: KamalanathanN <31615486+KamalanathanN@users.noreply.github.com>

File: ABBRobots/IRB120/irb120_ros2_gazebo/urdf/irb120_macro.urdf.xacro (robot description, xacro)
@@ -77,5 +77,5 @@
         <origin xyz="0 0 0" rpy="0 0 0"/>
         <geometry>
-          <mesh filename="file://$(find irb120_ros2_gazebo)/meshes/visual/base_link.stl"/>
+          <mesh filename="file://$(find irb120_ros2_gazebo)/meshes/visual/base_link.dae"/>
         </geometry>
         <xacro:material_abb_orange />
@@ -99,5 +99,5 @@
         <origin xyz="0 0 0" rpy="0 0 0"/>
         <geometry>
-          <mesh filename="file://$(find irb120_ros2_gazebo)/meshes/visual/link_1.stl"/>
+          <mesh filename="file://$(find irb120_ros2_gazebo)/meshes/visual/link_1.dae"/>
         </geometry>
         <xacro:material_abb_orange />
@@ -121,5 +121,5 @@
         <origin xyz="0 0 0" rpy="0 0 0"/>
         <geometry>
-          <mesh filename="file://$(find irb120_ros2_gazebo)/meshes/visual/link_2.stl"/>
+          <mesh filename="file://$(find irb120_ros2_gazebo)/meshes/visual/link_2.dae"/>
         </geometry>
         <xacro:material_abb_orange />
@@ -143,5 +143,5 @@
         <origin xyz="0 0 0" rpy="0 0 0"/>
         <geometry>
-          <mesh filename="file://$(find irb120_ros2_gazebo)/meshes/visual/link_3.stl"/>
+          <mesh filename="file://$(find irb120_ros2_gazebo)/meshes/visual/link_3.dae"/>
         </geometry>
         <xacro:material_abb_orange />
@@ -165,5 +165,5 @@
         <origin xyz="0 0 0" rpy="0 0 0"/>
         <geometry>
-          <mesh filename="file://$(find irb120_ros2_gazebo)/meshes/visual/link_4.stl"/>
+          <mesh filename="file://$(find irb120_ros2_gazebo)/meshes/visual/link_4.dae"/>
         </geometry>
         <xacro:material_abb_orange />
@@ -187,5 +187,5 @@
         <origin xyz="0 0 0" rpy="0 0 0"/>
         <geometry>
-          <mesh filename="file://$(find irb120_ros2_gazebo)/meshes/visual/link_5.stl"/>
+          <mesh filename="file://$(find irb120_ros2_gazebo)/meshes/visual/link_5.dae"/>
         </geometry>
         <xacro:material_abb_orange />
@@ -209,5 +209,5 @@
         <origin xyz="0 0 0" rpy="0 0 0"/>
         <geometry>
-          <mesh filename="file://$(find irb120_ros2_gazebo)/meshes/visual/link_6.stl"/>
+          <mesh filename="file://$(find irb120_ros2_gazebo)/meshes/visual/link_6.dae"/>
         </geometry>
         <xacro:material_abb_black />
