Commit message: Tidy up code: ABB IRB1200.

File: ABBRobots/IRB1200/irb1200_ros2_gazebo/urdf/irb1200.urdf.xacro (robot description, xacro)
@@ -48,12 +48,27 @@
 -->
 <robot name="irb1200" xmlns:xacro="http://ros.org/wiki/xacro">
+  <!-- ===== ARGUMENTS ===== -->
+  <!-- CELL LAYOUT:  -->
+  <xacro:arg name="cell_layout_1" default="false"/>
+  <xacro:property name="cell_layout_1" value="$(arg cell_layout_1)"/>
+  <!-- END-EFFECTOR:  -->
+  <xacro:arg name="EE_no" default="false"/>
+  <xacro:property name="EE_no" value="$(arg EE_no)"/>
   <!-- Include XACRO-MACRO file of the IRB1200: -->
   <xacro:include filename="$(find irb1200_ros2_gazebo)/urdf/irb1200_macro.urdf.xacro"/>
-  <xacro:irb1200 prefix=""/>
-  <!-- Fix robot to Gazebo world -->
+  <xacro:irb1200
+    prefix=""
+    EE_no="${EE_no}"
+  />
+  <!-- Gazebo world link: -->
   <link name="world"/>
-  <joint name="world-base_link-fixed" type="fixed">
-    <parent link="world"/>
-    <child link="base_link"/>
-  </joint>
+  <!-- ========== ========== ========== ========== ========== ========== -->
+  <!-- CELL LAYOUT SELECTION: -->
+  <!-- CELL LAYOUT N1) ABB IRB120 Robot alone: -->
+  <xacro:if value="${cell_layout_1}">
+    <joint name="world-base_link-fixed" type="fixed">
+      <parent link="world"/>
+      <child link="base_link"/>
+    </joint>
+  </xacro:if>
 </robot>

File: ABBRobots/IRB1200/irb1200_ros2_gazebo/urdf/irb1200_macro.urdf.xacro (robot description, xacro)
@@ -50,16 +50,19 @@
   <!-- Include additional ABB-Resources/MATERIALS+COLOUR xacro files: -->
   <xacro:include filename="$(find irb1200_ros2_gazebo)/urdf/abb_resources/common_materials.xacro"/>
-  <!-- Load TRANSMISSION file: -->
-  <xacro:include filename="$(find irb1200_ros2_gazebo)/urdf/irb1200_transmission.xacro" />
-  <!-- Load GAZEBO/ROS2_CONTROL file: -->
-  <xacro:include filename="$(find irb1200_ros2_gazebo)/urdf/irb1200_gazebo.xacro" />
   <!-- XACRO-MACRO of ABB-IRB1200: -->
-  <xacro:macro name="irb1200" params="prefix">
-    <!-- ABB-IRB1200 TRANSMISSION: -->
-    <xacro:irb1200_transmission prefix=""/>
-    <!-- ABB-IRB1200 GAZEBO - ROS2_CONTROL: -->
-    <xacro:irb1200_gazebo prefix=""/>
+  <xacro:macro name="irb1200" params="prefix EE_no">
+    <!-- Load ABB IRB1200 TRANSMISSION file: -->
+    <xacro:include filename="$(find irb1200_ros2_gazebo)/urdf/irb1200_transmission.xacro" />
+    <xacro:irb1200_transmission
+      prefix=""
+    />
+    <!-- Load ABB IRB1200 ROS2_CONTROL file: -->
+    <xacro:include filename="$(find irb1200_ros2_gazebo)/urdf/irb1200_ros2control.xacro" />
+    <xacro:irb1200_ros2control
+      prefix=""
+      EE_no="${EE_no}"
+    />
     <!-- ***** ABB-IRB1200 ROBOT .urdf SERIAL CHAIN ***** -->
-    <!-- ===== LINK LIST ===== -->
+    <!-- Link list: -->
     <!-- base_link -->
     <link name="${prefix}base_link">
@@ -210,5 +213,5 @@
     </link>
     <!-- end of link list -->
-    <!-- ===== JOINT LIST ===== -->
+    <!-- Joint list: -->
     <!-- joint_1 -->
     <joint type="revolute" name="${prefix}joint_1">

File: ABBRobots/IRB1200/irb1200_ros2_gazebo/urdf/irb1200_ros2control.xacro (robot description, xacro)
@@ -48,12 +48,19 @@
 -->
 <robot xmlns:xacro="http://www.ros.org/wiki/xacro">
-  <xacro:macro name="irb1200_gazebo" params="prefix" >
-    <gazebo>
-      <plugin filename="libgazebo_ros2_control.so" name="gazebo_ros2_control">
-        <robot_sim_type>gazebo_ros2_control/GazeboSystem</robot_sim_type>
-        <parameters>$(find irb1200_ros2_gazebo)/config/irb1200_controller.yaml</parameters>
-      </plugin>
-    </gazebo>
-    <ros2_control name="GazeboSystem" type="system">
+  <xacro:macro name="irb1200_ros2control" params="prefix EE_no" >
+    <!-- ROS2_CONTROL tag name: -->
+    <xacro:property name="name" value="GazeboSystem"/>
+    <!-- ===== Gazebo ROS2_CONTROL plugin ===== -->
+    <!-- No End-Effector: -->
+    <xacro:if value="${EE_no}">
+      <gazebo>
+        <plugin filename="libgazebo_ros2_control.so" name="gazebo_ros2_control">
+          <robot_sim_type>gazebo_ros2_control/GazeboSystem</robot_sim_type>
+          <parameters>$(find irb1200_ros2_gazebo)/config/irb1200_controller.yaml</parameters>
+        </plugin>
+      </gazebo>
+    </xacro:if>
+    <!-- ========== ROS2 CONTROL ========== -->
+    <ros2_control name="${name}" type="system">
       <hardware>
         <plugin>gazebo_ros2_control/GazeboSystem</plugin>
