Commit message: Tidy up code: ABB IRB6640.

File: ABBRobots/IRB6640/irb6640_ros2_gazebo/urdf/irb6640.urdf.xacro (robot description, xacro)
@@ -48,12 +48,27 @@
 -->
 <robot name="irb6640" xmlns:xacro="http://ros.org/wiki/xacro">
-  <!-- Include XACRO-MACRO file of the irb6640: -->
+  <!-- ===== ARGUMENTS ===== -->
+  <!-- CELL LAYOUT:  -->
+  <xacro:arg name="cell_layout_1" default="false"/>
+  <xacro:property name="cell_layout_1" value="$(arg cell_layout_1)"/>
+  <!-- END-EFFECTOR:  -->
+  <xacro:arg name="EE_no" default="false"/>
+  <xacro:property name="EE_no" value="$(arg EE_no)"/>
+  <!-- Include XACRO-MACRO file of the IRB6640: -->
   <xacro:include filename="$(find irb6640_ros2_gazebo)/urdf/irb6640_macro.urdf.xacro"/>
-  <xacro:irb6640 prefix=""/>
-  <!-- Fix robot to Gazebo world -->
+  <xacro:irb6640
+    prefix=""
+    EE_no="${EE_no}"
+  />
+  <!-- Gazebo world link: -->
   <link name="world"/>
-  <joint name="world-irb6640-fixed" type="fixed">
-    <parent link="world"/>
-    <child link="base_link"/>
-  </joint>
+  <!-- ========== ========== ========== ========== ========== ========== -->
+  <!-- CELL LAYOUT SELECTION: -->
+  <!-- CELL LAYOUT N1) ABB IRB6640 Robot alone: -->
+  <xacro:if value="${cell_layout_1}">
+    <joint name="world-base_link-fixed" type="fixed">
+      <parent link="world"/>
+      <child link="base_link"/>
+    </joint>
+  </xacro:if>
 </robot>

File: ABBRobots/IRB6640/irb6640_ros2_gazebo/urdf/irb6640_macro.urdf.xacro (robot description, xacro)
@@ -50,14 +50,17 @@
   <!-- Include additional ABB-Resources/MATERIALS+COLOUR xacro files: -->
   <xacro:include filename="$(find irb6640_ros2_gazebo)/urdf/abb_resources/common_materials.xacro"/>
-  <!-- Load TRANSMISSION file: -->
-  <xacro:include filename="$(find irb6640_ros2_gazebo)/urdf/irb6640_transmission.xacro" />
-  <!-- Load GAZEBO/ROS2_CONTROL file: -->
-  <xacro:include filename="$(find irb6640_ros2_gazebo)/urdf/irb6640_gazebo.xacro" />
-  <!-- XACRO-MACRO of ABB-irb6640: -->
-  <xacro:macro name="irb6640" params="prefix">
-    <!-- ABB-irb6640 TRANSMISSION: -->
-    <xacro:irb6640_transmission prefix=""/>
-    <!-- ABB-irb6640 GAZEBO - ROS2_CONTROL: -->
-    <xacro:irb6640_gazebo prefix=""/>
+  <!-- XACRO-MACRO of ABB-IRB6640: -->
+  <xacro:macro name="irb6640" params="prefix EE_no">
+    <!-- Load ABB IRB6640 TRANSMISSION file: -->
+    <xacro:include filename="$(find irb6640_ros2_gazebo)/urdf/irb6640_transmission.xacro" />
+    <xacro:irb6640_transmission
+      prefix=""
+    />
+    <!-- Load ABB IRB6640 ROS2_CONTROL file: -->
+    <xacro:include filename="$(find irb6640_ros2_gazebo)/urdf/irb6640_ros2control.xacro" />
+    <xacro:irb6640_ros2control
+      prefix=""
+      EE_no="${EE_no}"
+    />
     <!-- ***** ABB-irb6640 ROBOT .urdf SERIAL CHAIN ***** -->
     <!-- Due to the absence of data (specifications) in the official ABB ROS repositories,

File: ABBRobots/IRB6640/irb6640_ros2_gazebo/urdf/irb6640_ros2control.xacro (robot description, xacro)
@@ -48,12 +48,19 @@
 -->
 <robot xmlns:xacro="http://www.ros.org/wiki/xacro">
-  <xacro:macro name="irb6640_gazebo" params="prefix" >
-    <gazebo>
-      <plugin filename="libgazebo_ros2_control.so" name="gazebo_ros2_control">
-        <robot_sim_type>gazebo_ros2_control/GazeboSystem</robot_sim_type>
-        <parameters>$(find irb6640_ros2_gazebo)/config/irb6640_controller.yaml</parameters>
-      </plugin>
-    </gazebo>
-    <ros2_control name="GazeboSystem" type="system">
+  <xacro:macro name="irb6640_ros2control" params="prefix EE_no" >
+    <!-- ROS2_CONTROL tag name: -->
+    <xacro:property name="name" value="GazeboSystem"/>
+    <!-- ===== Gazebo ROS2_CONTROL plugin ===== -->
+    <!-- No End-Effector: -->
+    <xacro:if value="${EE_no}">
+      <gazebo>
+        <plugin filename="libgazebo_ros2_control.so" name="gazebo_ros2_control">
+          <robot_sim_type>gazebo_ros2_control/GazeboSystem</robot_sim_type>
+          <parameters>$(find irb6640_ros2_gazebo)/config/irb6640_controller.yaml</parameters>
+        </plugin>
+      </gazebo>
+    </xacro:if>
+    <!-- ========== ROS2 CONTROL ========== -->
+    <ros2_control name="${name}" type="system">
       <hardware>
         <plugin>gazebo_ros2_control/GazeboSystem</plugin>
