Commit message: Tidy up code: Fanuc CR35-iA.

File: Fanuc/CR35iA/cr35ia_ros2_gazebo/urdf/cr35ia.urdf.xacro (robot description, xacro)
@@ -47,12 +47,27 @@
 -->
 <robot name="cr35ia" xmlns:xacro="http://ros.org/wiki/xacro">
-  <!-- Include XACRO-MACRO file of the CR35iA: -->
+  <!-- ===== ARGUMENTS ===== -->
+  <!-- CELL LAYOUT:  -->
+  <xacro:arg name="cell_layout_1" default="false"/>
+  <xacro:property name="cell_layout_1" value="$(arg cell_layout_1)"/>
+  <!-- END-EFFECTOR:  -->
+  <xacro:arg name="EE_no" default="false"/>
+  <xacro:property name="EE_no" value="$(arg EE_no)"/>
+  <!-- Include XACRO-MACRO file of the cr35ia: -->
   <xacro:include filename="$(find cr35ia_ros2_gazebo)/urdf/cr35ia_macro.urdf.xacro"/>
-  <xacro:cr35ia prefix=""/>
-  <!-- Fix robot to Gazebo world -->
+  <xacro:cr35ia
+    prefix=""
+    EE_no="${EE_no}"
+  />
+  <!-- Gazebo world link: -->
   <link name="world"/>
-  <joint name="world-base_link-fixed" type="fixed">
-    <parent link="world"/>
-    <child link="base_link"/>
-  </joint>
+  <!-- ========== ========== ========== ========== ========== ========== -->
+  <!-- CELL LAYOUT SELECTION: -->
+  <!-- CELL LAYOUT N1) Fanuc CR35-iA Robot alone: -->
+  <xacro:if value="${cell_layout_1}">
+    <joint name="world-base_link-fixed" type="fixed">
+      <parent link="world"/>
+      <child link="base_link"/>
+    </joint>
+  </xacro:if>
 </robot>

File: Fanuc/CR35iA/cr35ia_ros2_gazebo/urdf/cr35ia_macro.urdf.xacro (robot description, xacro)
@@ -49,14 +49,17 @@
   <!-- Include additional FANUC-materials xacro files: -->
   <!-- <xacro:include filename="$(find cr35ia_ros2_gazebo)/urdf/fanuc_resources/common_materials.xacro" /> -->
-  <!-- Load TRANSMISSION file: -->
-  <xacro:include filename="$(find cr35ia_ros2_gazebo)/urdf/cr35ia_transmission.xacro" />
-  <!-- Load GAZEBO/ROS2_CONTROL file: -->
-  <xacro:include filename="$(find cr35ia_ros2_gazebo)/urdf/cr35ia_gazebo.xacro" />
-  <!-- XACRO-MACRO of FANUC CR35-iA: -->
-  <xacro:macro name="cr35ia" params="prefix">
-    <!-- FANUC CR35-iA TRANSMISSION: -->
-    <xacro:cr35ia_transmission prefix=""/>
-    <!-- FANUC CR35-iA GAZEBO - ROS2_CONTROL: -->
-    <xacro:cr35ia_gazebo prefix=""/>
+  <!-- XACRO-MACRO of Fanuc CR35-iA: -->
+  <xacro:macro name="cr35ia" params="prefix EE_no">
+    <!-- Load Fanuc CR35-iA TRANSMISSION file: -->
+    <xacro:include filename="$(find cr35ia_ros2_gazebo)/urdf/cr35ia_transmission.xacro" />
+    <xacro:cr35ia_transmission
+      prefix=""
+    />
+    <!-- Load Fanuc CR35-iA ROS2_CONTROL file: -->
+    <xacro:include filename="$(find cr35ia_ros2_gazebo)/urdf/cr35ia_ros2control.xacro" />
+    <xacro:cr35ia_ros2control
+      prefix=""
+      EE_no="${EE_no}"
+    />
     <!-- ***** FANUC CR35-iA ROBOT .urdf SERIAL CHAIN ***** -->
     <!--

File: Fanuc/CR35iA/cr35ia_ros2_gazebo/urdf/cr35ia_ros2control.xacro (robot description, xacro)
@@ -47,12 +47,19 @@
 -->
 <robot xmlns:xacro="http://www.ros.org/wiki/xacro">
-  <xacro:macro name="cr35ia_gazebo" params="prefix" >
-    <gazebo>
-      <plugin filename="libgazebo_ros2_control.so" name="gazebo_ros2_control">
-        <robot_sim_type>gazebo_ros2_control/GazeboSystem</robot_sim_type>
-        <parameters>$(find cr35ia_ros2_gazebo)/config/cr35ia_controller.yaml</parameters>
-      </plugin>
-    </gazebo>
-    <ros2_control name="GazeboSystem" type="system">
+  <xacro:macro name="cr35ia_ros2control" params="prefix EE_no" >
+    <!-- ROS2_CONTROL tag name: -->
+    <xacro:property name="name" value="GazeboSystem"/>
+    <!-- ===== Gazebo ROS2_CONTROL plugin ===== -->
+    <!-- No End-Effector: -->
+    <xacro:if value="${EE_no}">
+      <gazebo>
+        <plugin filename="libgazebo_ros2_control.so" name="gazebo_ros2_control">
+          <robot_sim_type>gazebo_ros2_control/GazeboSystem</robot_sim_type>
+          <parameters>$(find cr35ia_ros2_gazebo)/config/cr35ia_controller.yaml</parameters>
+        </plugin>
+      </gazebo>
+    </xacro:if>
+    <!-- ========== ROS2 CONTROL ========== -->
+    <ros2_control name="${name}" type="system">
       <hardware>
         <plugin>gazebo_ros2_control/GazeboSystem</plugin>
