Commit message: Tidy up code: KUKA LBR-iiwa.

File: Kuka/LBRiiwa/iiwa_ros2_gazebo/urdf/iiwa.urdf.xacro (robot description, xacro)
@@ -48,43 +48,67 @@
 -->
 <robot name="iiwa" xmlns:xacro="http://ros.org/wiki/xacro">
-  <!-- Include XACRO-MACRO file of the KUKA LBR-IIWA: -->
+  <!-- ===== ARGUMENTS ===== -->
+  <!-- CELL LAYOUT:  -->
+  <xacro:arg name="cell_layout_1" default="false"/>
+  <xacro:property name="cell_layout_1" value="$(arg cell_layout_1)"/>
+  <xacro:arg name="cell_layout_2" default="false"/>
+  <xacro:property name="cell_layout_2" value="$(arg cell_layout_2)"/>
+  <!-- END-EFFECTOR:  -->
+  <xacro:arg name="EE_no" default="false"/>
+  <xacro:property name="EE_no" value="$(arg EE_no)"/>
+  <!-- Include XACRO-MACRO file of the KUKA LBR-iiwa: -->
   <xacro:include filename="$(find iiwa_ros2_gazebo)/urdf/iiwa_macro.urdf.xacro"/>
-  <xacro:iiwa prefix=""/>
-  <!-- Fix robot to Gazebo world -->
+  <xacro:iiwa
+    prefix=""
+    EE_no="${EE_no}"
+  />
+  <!-- Gazebo world link: -->
   <link name="world"/>
+  <!-- ========== ========== ========== ========== ========== ========== -->
+  <!-- CELL LAYOUT SELECTION: -->
+  <!-- CELL LAYOUT N1) KUKA LBR-iiwa Robot alone: -->
+  <xacro:if value="${cell_layout_1}">
+    <joint name="world-base_link-fixed" type="fixed">
+      <parent link="world"/>
+      <child link="base_link"/>
+    </joint>
+  </xacro:if>
+  <!-- CELL LAYOUT N2) KUKA LBR-iiwa Robot on top of a pedestal: -->
+  <xacro:if value="${cell_layout_2}">
     <link name='iiwa_base'>
-    <inertial>
-      <origin xyz="0 0 0" rpy="0 0 0"/>
-      <mass value="100"/>
-      <inertia ixx="0.01"  ixy="0"  ixz="0" iyy="0.01" iyz="0" izz="0.01" />
-    </inertial>
-    <collision name='collision'>
-      <origin xyz="0 0 0" rpy=" 0 0 0"/>
-      <geometry>
-        <box size = "0.2 0.2 1.3"/>
-      </geometry>
-    </collision>
-    <visual name='chassis_visual'>
-      <origin xyz="0 0 0" rpy=" 0 0 0"/>
-      <geometry>
-        <box size = "0.2 0.2 1.3"/>
-      </geometry>
-      <material name="red">
-        <color rgba="1 0 0 1"/>
-      </material>
-    </visual>
-  </link>
-  <gazebo reference="iiwa_base">
-    <material>Gazebo/Red</material>
-  </gazebo>
-  <joint name="world_joint" type="fixed">
-    <parent link="world" />
-    <child link = "iiwa_base" />
-    <origin xyz="0.0 0.0 0.65" rpy="0.0 0.0 0.0" />
-  </joint>
-  <joint name="ur_joint" type="fixed">
-    <parent link="iiwa_base" />
-    <child link = "base_link" />
-    <origin xyz="0.0 0.0 0.655" rpy="0.0 0.0 0.0" />
-  </joint>
+      <inertial>
+        <origin xyz="0 0 0" rpy="0 0 0"/>
+        <mass value="100"/>
+        <inertia ixx="0.01"  ixy="0"  ixz="0" iyy="0.01" iyz="0" izz="0.01" />
+      </inertial>
+      <collision name='collision'>
+        <origin xyz="0 0 0" rpy=" 0 0 0"/>
+        <geometry>
+          <box size = "0.2 0.2 1.3"/>
+        </geometry>
+      </collision>
+      <visual name='chassis_visual'>
+        <origin xyz="0 0 0" rpy=" 0 0 0"/>
+        <geometry>
+          <box size = "0.2 0.2 1.3"/>
+        </geometry>
+        <material name="red">
+          <color rgba="1 0 0 1"/>
+        </material>
+      </visual>
+    </link>
+    <gazebo reference="iiwa_base">
+      <material>Gazebo/Red</material>
+    </gazebo>
+    <joint name="world_joint" type="fixed">
+      <parent link="world" />
+      <child link = "iiwa_base" />
+      <origin xyz="0.0 0.0 0.65" rpy="0.0 0.0 0.0" />
+    </joint>
+    <joint name="iiwa_joint" type="fixed">
+      <parent link="iiwa_base" />
+      <child link = "base_link" />
+      <origin xyz="0.0 0.0 0.655" rpy="0.0 0.0 0.0" />
+    </joint>
+  </xacro:if>
 </robot>

File: Kuka/LBRiiwa/iiwa_ros2_gazebo/urdf/iiwa_macro.urdf.xacro (robot description, xacro)
@@ -48,16 +48,17 @@
 -->
 <robot xmlns:xacro="http://ros.org/wiki/xacro">
-  <!-- Include additional FANUC-materials xacro files: -->
-  <!-- <xacro:include filename="$(find iiwa_ros2_gazebo)/urdf/fanuc_resources/common_materials.xacro" /> -->
-  <!-- Load TRANSMISSION file: -->
-  <xacro:include filename="$(find iiwa_ros2_gazebo)/urdf/iiwa_transmission.xacro" />
-  <!-- Load GAZEBO/ROS2_CONTROL file: -->
-  <xacro:include filename="$(find iiwa_ros2_gazebo)/urdf/iiwa_gazebo.xacro" />
-  <!-- XACRO-MACRO of KUKA LBR-IIWA: -->
-  <xacro:macro name="iiwa" params="prefix">
-    <!-- KUKA LBR-IIWA TRANSMISSION: -->
-    <xacro:iiwa_transmission prefix=""/>
-    <!-- KUKA LBR-IIWA GAZEBO - ROS2_CONTROL: -->
-    <xacro:iiwa_gazebo prefix=""/>
+  <!-- XACRO-MACRO of FANUC LBR-iiwa: -->
+  <xacro:macro name="iiwa" params="prefix EE_no">
+    <!-- Load FANUC LBR-iiwa TRANSMISSION file: -->
+    <xacro:include filename="$(find iiwa_ros2_gazebo)/urdf/iiwa_transmission.xacro" />
+    <xacro:iiwa_transmission
+      prefix=""
+    />
+    <!-- Load FANUC LBR-iiwa ROS2_CONTROL file: -->
+    <xacro:include filename="$(find iiwa_ros2_gazebo)/urdf/iiwa_ros2control.xacro" />
+    <xacro:iiwa_ros2control
+      prefix=""
+      EE_no="${EE_no}"
+    />
     <!-- ***** KUKA LBR-IIWA ROBOT .urdf SERIAL CHAIN ***** -->
     <!--

File: Kuka/LBRiiwa/iiwa_ros2_gazebo/urdf/iiwa_ros2control.xacro (robot description, xacro)
@@ -48,12 +48,19 @@
 -->
 <robot xmlns:xacro="http://www.ros.org/wiki/xacro">
-  <xacro:macro name="iiwa_gazebo" params="prefix" >
-    <gazebo>
-      <plugin filename="libgazebo_ros2_control.so" name="gazebo_ros2_control">
-        <robot_sim_type>gazebo_ros2_control/GazeboSystem</robot_sim_type>
-        <parameters>$(find iiwa_ros2_gazebo)/config/iiwa_controller.yaml</parameters>
-      </plugin>
-    </gazebo>
-    <ros2_control name="GazeboSystem" type="system">
+  <xacro:macro name="iiwa_ros2control" params="prefix EE_no" >
+    <!-- ROS2_CONTROL tag name: -->
+    <xacro:property name="name" value="GazeboSystem"/>
+    <!-- ===== Gazebo ROS2_CONTROL plugin ===== -->
+    <!-- No End-Effector: -->
+    <xacro:if value="${EE_no}">
+      <gazebo>
+        <plugin filename="libgazebo_ros2_control.so" name="gazebo_ros2_control">
+          <robot_sim_type>gazebo_ros2_control/GazeboSystem</robot_sim_type>
+          <parameters>$(find iiwa_ros2_gazebo)/config/iiwa_controller.yaml</parameters>
+        </plugin>
+      </gazebo>
+    </xacro:if>
+    <!-- ========== ROS2 CONTROL ========== -->
+    <ros2_control name="${name}" type="system">
       <hardware>
         <plugin>gazebo_ros2_control/GazeboSystem</plugin>
