Commit message: Tidy up code: Panda Robot.

File: PandaRobot/panda_ros2_gazebo/urdf/panda.urdf.xacro (robot description, xacro)
@@ -47,44 +47,67 @@
 -->
 <robot xmlns:xacro="http://wiki.ros.org/xacro" name="panda">
-  <!-- Include XACRO-MACRO FILE OF THE PANDA ROBOT -->
-  <xacro:include filename="$(find panda_ros2_gazebo)/urdf/panda_macro.urdf.xacro" />
-  <!-- Initialise PANDA ROBOT .urdf -->
-  <xacro:panda_robot/>
+  <!-- ===== ARGUMENTS ===== -->
+  <!-- CELL LAYOUT:  -->
+  <xacro:arg name="cell_layout_1" default="false"/>
+  <xacro:property name="cell_layout_1" value="$(arg cell_layout_1)"/>
+  <xacro:arg name="cell_layout_2" default="false"/>
+  <xacro:property name="cell_layout_2" value="$(arg cell_layout_2)"/>
+  <!-- END-EFFECTOR:  -->
+  <xacro:arg name="EE_no" default="false"/>
+  <xacro:property name="EE_no" value="$(arg EE_no)"/>
+  <!-- Include XACRO-MACRO file of the PANDA ROBOT: -->
+  <xacro:include filename="$(find panda_ros2_gazebo)/urdf/panda_macro.urdf.xacro"/>
+  <xacro:panda
+    prefix=""
+    EE_no="${EE_no}"
+  />
+  <!-- Gazebo world link: -->
   <link name="world"/>
-  <!-- <link name='panda_base'>
-    <inertial>
-      <origin xyz="0 0 0" rpy="0 0 0"/>
-      <mass value="100"/>
-      <inertia ixx="0.01"  ixy="0"  ixz="0" iyy="0.01" iyz="0" izz="0.01" />
-    </inertial>
-    <collision name='collision'>
-      <origin xyz="0 0 0" rpy=" 0 0 0"/>
-      <geometry>
-        <box size = "0.2 0.2 1.3"/>
-      </geometry>
-    </collision>
-    <visual name='chassis_visual'>
-      <origin xyz="0 0 0" rpy=" 0 0 0"/>
-      <geometry>
-        <box size = "0.2 0.2 1.3"/>
-      </geometry>
-      <material name="red">
-        <color rgba="1 0 0 1"/>
-      </material>
-    </visual>
-  </link>
-  <gazebo reference="panda_base">
-    <material>Gazebo/Red</material>
-  </gazebo> -->
-  <joint name="world_joint" type="fixed">
-    <parent link="world" />
-    <!-- <child link = "panda_base" /> -->
-    <child link = "panda_link0" />
-    <origin xyz="0.0 0.0 0.0" rpy="0.0 0.0 0.0" /> <!-- <origin xyz="0.0 0.0 0.65" rpy="0.0 0.0 0.0" /> -->
-  </joint>
-  <!-- <joint name="panda_joint" type="fixed">
-    <parent link="panda_base" />
-    <child link = "panda_link0" />
-    <origin xyz="0.05 0.0 0.65" rpy="0.0 0.0 0.0" />
-  </joint> -->
+  <!-- ========== ========== ========== ========== ========== ========== -->
+  <!-- CELL LAYOUT SELECTION: -->
+  <!-- CELL LAYOUT N1) PANDA ROBOT alone: -->
+  <xacro:if value="${cell_layout_1}">
+    <joint name="world-base_link-fixed" type="fixed">
+      <parent link="world"/>
+      <child link="panda_link0"/>
+    </joint>
+  </xacro:if>
+  <!-- CELL LAYOUT N2) PANDA ROBOT on top of a pedestal: -->
+  <xacro:if value="${cell_layout_2}">
+    <link name='panda_base'>
+      <inertial>
+        <origin xyz="0 0 0" rpy="0 0 0"/>
+        <mass value="100"/>
+        <inertia ixx="0.01"  ixy="0"  ixz="0" iyy="0.01" iyz="0" izz="0.01" />
+      </inertial>
+      <collision name='collision'>
+        <origin xyz="0 0 0" rpy=" 0 0 0"/>
+        <geometry>
+          <box size = "0.2 0.2 1.3"/>
+        </geometry>
+      </collision>
+      <visual name='chassis_visual'>
+        <origin xyz="0 0 0" rpy=" 0 0 0"/>
+        <geometry>
+          <box size = "0.2 0.2 1.3"/>
+        </geometry>
+        <material name="red">
+          <color rgba="1 0 0 1"/>
+        </material>
+      </visual>
+    </link>
+    <gazebo reference="panda_base">
+      <material>Gazebo/Red</material>
+    </gazebo>
+    <joint name="world_joint" type="fixed">
+      <parent link="world" />
+      <child link = "panda_base" />
+      <origin xyz="0.0 0.0 0.65" rpy="0.0 0.0 0.0" />
+    </joint>
+    <joint name="panda_joint" type="fixed">
+      <parent link="panda_base" />
+      <child link = "panda_link0" />
+      <origin xyz="0.0 0.0 0.655" rpy="0.0 0.0 0.0" />
+    </joint>
+  </xacro:if>
 </robot>

File: PandaRobot/panda_ros2_gazebo/urdf/panda_macro.urdf.xacro (robot description, xacro)
@@ -47,13 +47,17 @@
 -->
 <robot xmlns:xacro="http://wiki.ros.org/xacro">
-  <!-- Load TRANSMISSION file: -->
-  <xacro:include filename="$(find panda_ros2_gazebo)/urdf/panda_transmission.xacro" />
-  <!-- Load GAZEBO/ROS2_CONTROL file: -->
-  <xacro:include filename="$(find panda_ros2_gazebo)/urdf/panda_gazebo.xacro" />
-  <xacro:macro name="panda_robot">
-    <!-- PANDA TRANSMISSION: -->
-    <xacro:panda_transmission />
-    <!-- PANDA GAZEBO - ROS2_CONTROL: -->
-    <xacro:panda_gazebo />
+  <!-- XACRO-MACRO of PANDA ROBOT: -->
+  <xacro:macro name="panda" params="prefix EE_no">
+    <!-- Load PANDA ROBOT TRANSMISSION file: -->
+    <xacro:include filename="$(find panda_ros2_gazebo)/urdf/panda_transmission.xacro" />
+    <xacro:panda_transmission
+      prefix=""
+    />
+    <!-- Load PANDA ROBOT ROS2_CONTROL file: -->
+    <xacro:include filename="$(find panda_ros2_gazebo)/urdf/panda_ros2control.xacro" />
+    <xacro:panda_ros2control
+      prefix=""
+      EE_no="${EE_no}"
+    />
     <!-- ***** PANDA ROBOT .urdf SERIAL CHAIN ***** -->
     <!-- panda_link0 -->

File: PandaRobot/panda_ros2_gazebo/urdf/panda_ros2control.xacro (robot description, xacro)
@@ -47,12 +47,19 @@
 -->
 <robot xmlns:xacro="http://www.ros.org/wiki/xacro">
-  <xacro:macro name="panda_gazebo" >
-    <gazebo>
-      <plugin filename="libgazebo_ros2_control.so" name="gazebo_ros2_control">
-        <robot_sim_type>gazebo_ros2_control/GazeboSystem</robot_sim_type>
-        <parameters>$(find panda_ros2_gazebo)/config/panda_controller.yaml</parameters>
-      </plugin>
-    </gazebo>
-    <ros2_control name="GazeboSystem" type="system">
+  <xacro:macro name="panda_ros2control" params="prefix EE_no" >
+    <!-- ROS2_CONTROL tag name: -->
+    <xacro:property name="name" value="GazeboSystem"/>
+    <!-- ===== Gazebo ROS2_CONTROL plugin ===== -->
+    <!-- No End-Effector: -->
+    <xacro:if value="${EE_no}">
+      <gazebo>
+        <plugin filename="libgazebo_ros2_control.so" name="gazebo_ros2_control">
+          <robot_sim_type>gazebo_ros2_control/GazeboSystem</robot_sim_type>
+          <parameters>$(find panda_ros2_gazebo)/config/panda_controller.yaml</parameters>
+        </plugin>
+      </gazebo>
+    </xacro:if>
+    <!-- ========== ROS2 CONTROL ========== -->
+    <ros2_control name="${name}" type="system">
       <hardware>
         <plugin>gazebo_ros2_control/GazeboSystem</plugin>

File: PandaRobot/panda_ros2_gazebo/urdf/panda_transmission.xacro (robot description, xacro)
@@ -47,5 +47,5 @@
 -->
 <robot xmlns:xacro="http://wiki.ros.org/xacro">
-  <xacro:macro name="panda_transmission" >
+  <xacro:macro name="panda_transmission" params="prefix">
     <transmission name="panda_joint1_trans">
       <type>transmission_interface/SimpleTransmission</type>
