Commit message: Tidy up code: UR Robots.

File: UniversalRobots/UR5/ur5_ros2_gazebo/urdf/ur5.urdf.xacro (robot description, xacro)
@@ -55,56 +55,78 @@
 -->
 <robot xmlns:xacro="http://wiki.ros.org/xacro" name="ur5">
-    <!-- Include XACRO-MACRO FILE OF THE ur5 ROBOT -->
-    <xacro:include filename="$(find ur5_ros2_gazebo)/urdf/ur5_macro.urdf.xacro" />
-    <!-- Load and initialise ur5 INITIAL POSITIONS FILE:
-    <xacro:arg name="initial_positions_file" default="$(find ur5_ros2_gazebo/config/initial_positions.yaml"/>
-    <xacro:property name="initial_positions_file" default="$(arg initial_positions_file)"/> -->
-    <!-- IF ADD TO ur5_robot: initial_positions="${load_yaml(initial_positions_file)}" -->
-    <!-- Initialise PARAMS: -->
-    <xacro:arg name="safety_limits" default="false"/>
-    <xacro:arg name="safety_pos_margin" default="0.15"/>
-    <xacro:arg name="safety_k_position" default="20"/>
-    <!-- Initialise ur5 ROBOT .urdf -->
-    <xacro:ur5_robot
-        prefix = ""
-        safety_limits="$(arg safety_limits)"
-        safety_pos_margin="$(arg safety_pos_margin)"
-        safety_k_position="$(arg safety_k_position)"
-    />
-    <link name="world"/>
+  <!-- Load and initialise UR5 INITIAL POSITIONS FILE:
+  <xacro:arg name="initial_positions_file" default="$(find ur5_ros2_gazebo/config/initial_positions.yaml"/>
+  <xacro:property name="initial_positions_file" default="$(arg initial_positions_file)"/> -->
+  <!-- IF ADD TO UR5: initial_positions="${load_yaml(initial_positions_file)}" -->
+  <!-- ===== ARGUMENTS ===== -->
+  <!-- CELL LAYOUT:  -->
+  <xacro:arg name="cell_layout_1" default="false"/>
+  <xacro:property name="cell_layout_1" value="$(arg cell_layout_1)"/>
+  <xacro:arg name="cell_layout_2" default="false"/>
+  <xacro:property name="cell_layout_2" value="$(arg cell_layout_2)"/>
+  <!-- END-EFFECTOR:  -->
+  <xacro:arg name="EE_no" default="false"/>
+  <xacro:property name="EE_no" value="$(arg EE_no)"/>
+  <!-- UR Robot PARAMS: -->
+  <xacro:arg name="safety_limits" default="false"/>
+  <xacro:arg name="safety_pos_margin" default="0.15"/>
+  <xacro:arg name="safety_k_position" default="20"/>
+  <!-- Include XACRO-MACRO file of the UR5 ROBOT: -->
+  <xacro:include filename="$(find ur5_ros2_gazebo)/urdf/ur5_macro.urdf.xacro"/>
+  <xacro:ur5
+    prefix=""
+    EE_no="${EE_no}"
+    safety_limits="$(arg safety_limits)"
+    safety_pos_margin="$(arg safety_pos_margin)"
+    safety_k_position="$(arg safety_k_position)"
+  />
+  <!-- Gazebo world link: -->
+  <link name="world"/>
+  <!-- ========== ========== ========== ========== ========== ========== -->
+  <!-- CELL LAYOUT SELECTION: -->
+  <!-- CELL LAYOUT N1) UR5 ROBOT alone: -->
+  <xacro:if value="${cell_layout_1}">
+    <joint name="world-base_link-fixed" type="fixed">
+      <parent link="world"/>
+      <child link="base_link"/>
+    </joint>
+  </xacro:if>
+  <!-- CELL LAYOUT N2) UR5 ROBOT on top of a pedestal: -->
+  <xacro:if value="${cell_layout_2}">
     <link name='ur_base'>
-    <inertial>
-      <origin xyz="0 0 0" rpy="0 0 0"/>
-      <mass value="100"/>
-      <inertia ixx="0.01"  ixy="0"  ixz="0" iyy="0.01" iyz="0" izz="0.01" />
-    </inertial>
-    <collision name='collision'>
-      <origin xyz="0 0 0" rpy=" 0 0 0"/>
-      <geometry>
-        <box size = "0.2 0.2 1.3"/>
-      </geometry>
-    </collision>
-    <visual name='chassis_visual'>
-      <origin xyz="0 0 0" rpy=" 0 0 0"/>
-      <geometry>
-        <box size = "0.2 0.2 1.3"/>
-      </geometry>
-      <material name="red">
-        <color rgba="1 0 0 1"/>
-      </material>
-    </visual>
-  </link>
-  <gazebo reference="ur_base">
-    <material>Gazebo/Red</material>
-  </gazebo>
-  <joint name="world_joint" type="fixed">
-    <parent link="world" />
-    <child link = "ur_base" />
-    <origin xyz="0.0 0.0 0.65" rpy="0.0 0.0 0.0" />
-  </joint>
-  <joint name="ur_joint" type="fixed">
-    <parent link="ur_base" />
-    <child link = "base_link" />
-    <origin xyz="0.0 0.0 0.655" rpy="0.0 0.0 0.0" />
-  </joint>
+      <inertial>
+        <origin xyz="0 0 0" rpy="0 0 0"/>
+        <mass value="100"/>
+        <inertia ixx="0.01"  ixy="0"  ixz="0" iyy="0.01" iyz="0" izz="0.01" />
+      </inertial>
+      <collision name='collision'>
+        <origin xyz="0 0 0" rpy=" 0 0 0"/>
+        <geometry>
+          <box size = "0.2 0.2 1.3"/>
+        </geometry>
+      </collision>
+      <visual name='chassis_visual'>
+        <origin xyz="0 0 0" rpy=" 0 0 0"/>
+        <geometry>
+          <box size = "0.2 0.2 1.3"/>
+        </geometry>
+        <material name="red">
+          <color rgba="1 0 0 1"/>
+        </material>
+      </visual>
+    </link>
+    <gazebo reference="ur_base">
+      <material>Gazebo/Red</material>
+    </gazebo>
+    <joint name="world_joint" type="fixed">
+      <parent link="world" />
+      <child link = "ur_base" />
+      <origin xyz="0.0 0.0 0.65" rpy="0.0 0.0 0.0" />
+    </joint>
+    <joint name="ur_joint" type="fixed">
+      <parent link="ur_base" />
+      <child link = "base_link" />
+      <origin xyz="0.0 0.0 0.655" rpy="0.0 0.0 0.0" />
+    </joint>
+  </xacro:if>
 </robot>

File: UniversalRobots/UR5/ur5_ros2_gazebo/urdf/ur5_macro.urdf.xacro (robot description, xacro)
@@ -55,21 +55,20 @@
 -->
 <robot xmlns:xacro="http://wiki.ros.org/xacro">
-  <!-- Load PROPERTIES file: -->
-  <xacro:include filename="$(find ur5_ros2_gazebo)/urdf/ur5_common.xacro" />
-  <!-- Load TRANSMISSION file: -->
-  <xacro:include filename="$(find ur5_ros2_gazebo)/urdf/ur5_transmission.xacro" />
-  <!-- Load GAZEBO/ROS2_CONTROL file: -->
-  <xacro:include filename="$(find ur5_ros2_gazebo)/urdf/ur5_gazebo.xacro" />
-  <xacro:macro name="ur5_robot" params="
-    prefix
-    safety_limits
-    safety_pos_margin
-    safety_k_position" >
-    <!-- ur5 SPECIFICATIONS/PARAMETERS: -->
+  <!-- XACRO-MACRO of UR5 ROBOT: -->
+  <xacro:macro name="ur5" params="prefix EE_no safety_limits safety_pos_margin safety_k_position">
+    <!-- Load UR5 ROBOT TRANSMISSION file: -->
+    <xacro:include filename="$(find ur5_ros2_gazebo)/urdf/ur5_transmission.xacro" />
+    <xacro:ur5_transmission
+      prefix=""
+    />
+    <!-- Load UR5 ROBOT ROS2_CONTROL file: -->
+    <xacro:include filename="$(find ur5_ros2_gazebo)/urdf/ur5_ros2control.xacro" />
+    <xacro:ur5_ros2control
+      prefix=""
+      EE_no="${EE_no}"
+    />
+    <!-- Load UR5 SPECIFICATIONS file: -->
+    <xacro:include filename="$(find ur5_ros2_gazebo)/urdf/ur5_common.xacro" />
     <xacro:ur5_common/>
-    <!-- ur5 TRANSMISSION: -->
-    <xacro:ur5_transmission prefix="${prefix}"/>
-    <!-- ur5 GAZEBO - ROS2_CONTROL: -->
-    <xacro:ur5_gazebo prefix="${prefix}"/>
     <!-- ***** ur5 ROBOT .urdf SERIAL CHAIN *****-->
     <!-- Links: -->

File: UniversalRobots/UR5/ur5_ros2_gazebo/urdf/ur5_ros2control.xacro (robot description, xacro)
@@ -26,5 +26,5 @@
 # ===================================== COPYRIGHT ===================================== #
 #                                                                                       #
-#  Some of the information used to build the ROS2 UR3-Robot .urdf files in this ROS2    #
+#  Some of the information used to build the ROS2 UR5-Robot .urdf files in this ROS2    #
 #  repository has been taken from the following resources:                              #
 #       - Universal Robots ROS2 Description:                                            #
@@ -55,47 +55,22 @@
 -->
 <robot xmlns:xacro="http://www.ros.org/wiki/xacro">
-  <xacro:macro name="ur3_gazebo" params="prefix">
-    <gazebo>
-      <plugin filename="libgazebo_ros2_control.so" name="gazebo_ros2_control">
-        <robot_sim_type>gazebo_ros2_control/GazeboSystem</robot_sim_type>
-        <parameters>$(find ur3_ros2_gazebo)/config/ur3_controller.yaml</parameters>
-      </plugin>
-    </gazebo>
-    <ros2_control name="GazeboSystem" type="system">
+  <xacro:macro name="ur5_ros2control" params="prefix EE_no" >
+    <!-- ROS2_CONTROL tag name: -->
+    <xacro:property name="name" value="GazeboSystem"/>
+    <!-- ===== Gazebo ROS2_CONTROL plugin ===== -->
+    <!-- No End-Effector: -->
+    <xacro:if value="${EE_no}">
+      <gazebo>
+        <plugin filename="libgazebo_ros2_control.so" name="gazebo_ros2_control">
+          <robot_sim_type>gazebo_ros2_control/GazeboSystem</robot_sim_type>
+          <parameters>$(find ur5_ros2_gazebo)/config/ur5_controller.yaml</parameters>
+        </plugin>
+      </gazebo>
+    </xacro:if>
+    <!-- ========== ROS2 CONTROL ========== -->
+    <ros2_control name="${name}" type="system">
       <hardware>
         <plugin>gazebo_ros2_control/GazeboSystem</plugin>
       </hardware>
-      <!--
-      <hardware>
-        <xacro:if value="${use_fake_hardware}">
-          <plugin>fake_components/GenericSystem</plugin>
-          <param name="fake_sensor_commands">${fake_sensor_commands}</param>
-          <param name="state_following_offset">0.0</param>
-        </xacro:if>
-        <xacro:unless value="${use_fake_hardware}">
-          <plugin>ur_robot_driver/URPositionHardwareInterface</plugin>
-          <param name="robot_ip">${robot_ip}</param>
-          <param name="script_filename">${script_filename}</param>
-          <param name="output_recipe_filename">${output_recipe_filename}</param>
-          <param name="input_recipe_filename">${input_recipe_filename}</param>
-          <param name="headless_mode">0</param>
-          <param name="reverse_port">50001</param>
-          <param name="script_sender_port">50002</param>
-          <param name="tf_prefix">"${tf_prefix}"</param>
-          <param name="non_blocking_read">0</param>
-          <param name="servoj_gain">2000</param>
-          <param name="servoj_lookahead_time">0.03</param>
-          <param name="use_tool_communication">0</param>
-          <param name="kinematics/hash">${hash_kinematics}</param>
-          <param name="tool_voltage">0</param>
-          <param name="tool_parity">0</param>
-          <param name="tool_baud_rate">115200</param>
-          <param name="tool_stop_bits">1</param>
-          <param name="tool_rx_idle_chars">1.5</param>
-          <param name="tool_tx_idle_chars">3.5</param>
-          <param name="tool_device_name">/tmp/ttyUR</param>
-          <param name="tool_tcp_port">54321</param>
-        </xacro:unless>
-      </hardware> -->
       <joint name="${prefix}shoulder_pan_joint">
         <command_interface name="position">
@@ -146,6 +121,6 @@
         </command_interface>
         <command_interface name="velocity">
-          <param name="min">-6.28</param>
-          <param name="max">6.28</param>
+          <param name="min">-3.2</param>
+          <param name="max">3.2</param>
         </command_interface>
         <state_interface name="position"/>
@@ -160,6 +135,6 @@
         </command_interface>
         <command_interface name="velocity">
-          <param name="min">-6.28</param>
-          <param name="max">6.28</param>
+          <param name="min">-3.2</param>
+          <param name="max">3.2</param>
         </command_interface>
         <state_interface name="position"/>
@@ -174,6 +149,6 @@
         </command_interface>
         <command_interface name="velocity">
-          <param name="min">-6.28</param>
-          <param name="max">6.28</param>
+          <param name="min">-3.2</param>
+          <param name="max">3.2</param>
         </command_interface>
         <state_interface name="position"/>
@@ -182,13 +157,4 @@
         <!-- <param name="initial_position">${initial_positions['wrist_3_joint']}</param>   initial position for the FakeSystem -->
       </joint>
-      <!--
-      <sensor name="tcp_fts_sensor">
-        <state_interface name="force.x"/>
-        <state_interface name="force.y"/>
-        <state_interface name="force.z"/>
-        <state_interface name="torque.x"/>
-        <state_interface name="torque.y"/>
-        <state_interface name="torque.z"/>
-      </sensor> -->
     </ros2_control>
     <gazebo reference="${prefix}shoulder_link">
